File: pcb/spi-control/spi-control.kicad_pcb (KiCad board)
At the start: 4 copper layers, 81.2 x 61.6 mm, 37 parts, among them J1 USB_C_Receptacle_USB2.0_16P, J16 Conn_01x06_Pin, J17 Conn_01x06_Pin, J18 Conn_01x06_Pin, J19 Conn_01x06_Pin, J2 Conn_01x04_Pin, J20 Conn_01x06_Pin, J21 Conn_01x06_Pin, J22 Conn_01x06_Pin, J23 Conn_01x06_Pin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

Commit message: Finish pcb design
Parts:
- added H1: MountingHole, MountingHole:MountingHole_2.5mm, F.Cu at (38.9, 44.4)
- added H2: MountingHole, MountingHole:MountingHole_2.5mm, F.Cu at (38.9, 68.4)
- added H3: MountingHole, MountingHole:MountingHole_2.5mm, F.Cu at (90.7, 68.4)
- added H4: MountingHole, MountingHole:MountingHole_2.5mm, F.Cu at (90.7, 44.4)
- added R5: 5k1, Resistor_SMD:R_0402_1005Metric, F.Cu at (41.1, 71.9)
- added R6: 5k1, Resistor_SMD:R_0402_1005Metric, F.Cu at (39.0, 71.9)
- R1: value 10k -> 5k1
- moved R3 14.0 mm to (38.7, 81.2), turned to -90 degrees
- moved C11 13.6 mm to (33.5, 72.0), turned to 180 degrees
- moved R1 13.2 mm to (67.2, 68.1), turned to 0 degrees
- moved J2 13.0 mm to (68.8, 75.5), turned to -90 degrees
- moved C5 12.1 mm to (60.8, 66.3), turned to 90 degrees
- moved C3 12.1 mm to (72.3, 61.1), turned to 0 degrees
- moved C10 11.2 mm to (37.3, 81.3), turned to -90 degrees
- moved C2 11.0 mm to (69.2, 68.1)
- moved C12 10.7 mm to (30.4, 61.4), turned to 180 degrees
- moved C1 8.43 mm to (72.3, 62.6), turned to 0 degrees
- moved C4 8.30 mm to (62.7, 57.4), turned to 90 degrees
- moved R4 7.66 mm to (37.4, 75.6)
- moved C9 7.48 mm to (64.1, 57.4), turned to 90 degrees
- moved U3 4.90 mm to (32.3, 66.6)
- moved R2 3.92 mm to (70.4, 65.6), turned to 90 degrees
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Connections:
- U1 pad 30: unconnected-(U1-PA9-Pad30) -> /VBUS
- U1 pad 5: /XTALO -> /XTALI
- U1 pad 6: /XTALI -> /XTALO
Routing:
- net +3V3: track 0.00 -> 371.2 mm, vias 0 -> 14
- net GND: track 0.76 -> 353.5 mm, vias 1 -> 48
- net /CS2: track 0.00 -> 189.2 mm, vias 0 -> 3
- net /CS3: track 0.00 -> 178.6 mm, vias 0 -> 4
- net /CS5: track 0.00 -> 165.6 mm, vias 0 -> 2
- net /CS1: track 0.00 -> 159.4 mm, vias 0 -> 2
- net /CS4: track 0.00 -> 137.7 mm, vias 0 -> 3
- net /SCK3: track 0.00 -> 115.7 mm, vias 0 -> 2
- net /SCK2: track 0.00 -> 111.4 mm, vias 0 -> 1
- net /MOSI3: track 0.00 -> 110.4 mm, vias 0 -> 2
- net /MISO3: track 0.00 -> 110.0 mm, vias 0 -> 1
- net /SCK1: track 0.00 -> 99.9 mm
- net /MISO2: track 0.00 -> 98.7 mm, vias 0 -> 1
- net /MOSI2: track 0.00 -> 97.9 mm, vias 0 -> 1
- net /MOSI1: track 0.00 -> 96.7 mm
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- added copper zone on B.Cu, net GND
Other:
- outline, holes or cut-outs redrawn
- copper layers 4 -> 2
