File: pcb/spi-control/spi-control.kicad_sch (KiCad schematic)
At the start: 24 parts, among them J1 USB_C_Receptacle_USB2.0_16P, J2 Conn_01x04_Pin, U1 STM32F411CEUx, U2 SRV05-4, U3 AMS1117-3.3, Y1 16MHz

Commit message: Finish pcb design
Parts:
- added H1, H2, H3, H4: MountingHole, MountingHole:MountingHole_2.5mm, symbol Mechanical:MountingHole
- J2: now not fitted
Connections:
- net USB+: no longer J1.A5 (CC1), J1.A7 (D-), J1.B7 (D-), R4.1, U1.32 (PA11), U2.1 (IO1)
- net XTALI: now also U1.5 (PH0); no longer U1.6 (PH1)
- net XTALO: now also U1.6 (PH1); no longer U1.5 (PH0)
- new net: J1.A5 (CC1), R4.1
- new net USB-: J1.A7 (D-), J1.B7 (D-), U1.32 (PA11), U2.1 (IO1)
